File: ctrl-m.kicad_sch (KiCad schematic)
At the start: 33 parts, among them J1 USB_B, J10 Conn_01x04, J11 Conn_01x05, J12 Conn_01x04, J2 Conn_ARM_JTAG_SWD_10, J3 Conn_01x01, J4 Conn_01x01, J5 Conn_01x01, J6 Conn_01x01, J7 Conn_01x16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

Commit message: Enhancement: have unused pins ending on a pad #8
Also migrated to KiCAD 9
Parts:
- added J13: Conn_01x08, Connector_PinHeader_2.54mm:PinHeader_1x08_P2.54mm_Vertical, symbol Connector_Generic:Conn_01x08
Connections:
- net +3V3: now also J13.1 (Pin_1)
- net GND: now also J13.8 (Pin_8)
- net B13: now reaches U3.26 (PB13)
- net B13: now also J13.2 (Pin_2)
- net B14: now reaches U3.27 (PB14)
- net B14: now also J13.3 (Pin_3)
- net B15: now reaches U3.28 (PB15)
- net B15: now also J13.4 (Pin_4)
- net A8: now reaches U3.29 (PA8)
- net A8: now also J13.5 (Pin_5)
- net A9: now reaches U3.30 (PA9)
- net A9: now also J13.6 (Pin_6)
- net A10: now reaches U3.31 (PA10)
- net A10: now also J13.7 (Pin_7)
- no-connect marks 8 -> 2
Other:
- note added: "Free Pins"
